File: radio.sch (KiCad schematic (older format))
At the start: 0 parts

Commit message: clain up depth
Parts:
- added E1: ANT-433-SP, radio:XDCR_ANT-433-SP, symbol ANT-433-SP:ANT-433-SP
Connections:
- net labels added: ANT, GND
- wire segments 12 -> 23
Other:
- note added: "Antenna"
- note added: "CAS Bus"
- note added: "Radio"
Changed lines of the file:
@@
 $EndDescr
 $Sheet
-S 2650 1800 500  700
+S 1500 1000 500  700
 U 5E51D523
 F0 "RFM69HCW" 50
 F1 "../hardware-sch-blocks/RFM69HCW/RFM69HCW.sch" 50
-F2 "INT" I L 2650 1850 50
-F3 "ANT" I L 2650 1950 50
-F4 "RST" I L 2650 2050 50
-F5 "nSS" I L 2650 2150 50
-F6 "MISO" I L 2650 2250 50
-F7 "MOSI" I L 2650 2350 50
-F8 "SCK" I L 2650 2450 50
+F2 "INT" I L 1500 1050 50
+F3 "ANT" I L 1500 1150 50
+F4 "RST" I L 1500 1250 50
+F5 "nSS" I L 1500 1350 50
+F6 "MISO" I L 1500 1450 50
+F7 "MOSI" I L 1500 1550 50
+F8 "SCK" I L 1500 1650 50
 $EndSheet
 Wire Wire Line
-	2100 2450 2650 2450
+	950  1650 1500 1650
 Wire Wire Line
-	2100 2250 2650 2250
+	950  1450 1500 1450
 Wire Wire Line
-	2100 2350 2650 2350
+	950  1550 1500 1550
 Wire Wire Line
-	2100 2150 2650 2150
+	950  1350 1500 1350
 Wire Wire Line
-	2100 2050 2650 2050
+	950  1250 1500 1250
 Wire Wire Line
-	2100 1850 2650 1850
-Text Label 2100 1850 2    50   ~ 0
+	950  1050 1500 1050
+Text Label 950  1050 2    50   ~ 0
 IO_39
-Text Label 2100 2050 2    50   ~ 0
+Text Label 950  1250 2    50   ~ 0
 IO_38
-Text Label 2100 2150 2    50   ~ 0
+Text Label 950  1350 2    50   ~ 0
 SPI_nSS1
-Text Label 2100 2250 2    50   ~ 0
+Text Label 950  1450 2    50   ~ 0
 SPI_MISO
-Text Label 2100 2350 2    50   ~ 0
+Text Label 950  1550 2    50   ~ 0
 SPI_MOSI
-Text Label 2100 2450 2    50   ~ 0
+Text Label 950  1650 2    50   ~ 0
 SPI_SCK
 $Sheet
-S 7650 1250 1250 1900
+S 1700 2500 1250 1900
 U 5ED12D30
 F0 "CAS-bus" 50
 F1 "../hardware-sch-blocks/CAS_bus/CAS_bus.sch" 50
-F2 "INT1" I L 7650 1350 50
-F3 "INT3" I L 7650 1450 50
-F4 "INT5" I L 7650 1550 50
-F5 "I2C0_SCL" I L 7650 1650 50
-F6 "I2C1_SCL" I L 7650 1750 50
-F7 "INT7" I L 7650 1850 50
-F8 "SPI0_nSS1" I L 7650 1950 50
-F9 "SPI0_SCK" I L 7650 2050 50
-F10 "SPI0_MISO" I L 7650 2150 50
-F11 "SPI0_MOSI" I L 7650 2250 50
-F12 "INT2" I R 8900 1350 50
-F13 "INT4" I R 8900 1450 50
-F14 "INT6" I R 8900 1550 50
-F15 "I2C0_SDA" I R 8900 1650 50
-F16 "I2C1_SDA" I R 8900 1750 50
-F17 "INT8" I R 8900 1850 50
-F18 "SPI0_nSS2" I R 8900 1950 50
-F19 "SPI0_nSS3" I R 8900 2050 50
-F20 "SPI0_nSS4" I R 8900 2150 50
-F21 "SPI0_nSS5" I R 8900 2250 50
-F22 "SPI0_nSS6" I R 8900 2350 50
-F23 "SPI0_nSS7" I R 8900 2450 50
-F24 "SPI0_nSS8" I R 8900 2550 50
-F25 "SPIHS_SCK" I L 7650 2800 50
-F26 "SPIHS_MISO" I R 8900 2800 50
-F27 "SPIHS_MOSI" I L 7650 2900 50
-F28 "SPIHS_nSS1" I L 7650 3000 50
-F29 "SPIHS_nSS2" I R 8900 3000 50
+F2 "INT1" I L 1700 2600 50
+F3 "INT3" I L 1700 2700 50
+F4 "INT5" I L 1700 2800 50
+F5 "I2C0_SCL" I L 1700 2900 50
+F6 "I2C1_SCL" I L 1700 3000 50
+F7 "INT7" I L 1700 3100 50
+F8 "SPI0_nSS1" I L 1700 3200 50
+F9 "SPI0_SCK" I L 1700 3300 50
+F10 "SPI0_MISO" I L 1700 3400 50
+F11 "SPI0_MOSI" I L 1700 3500 50
+F12 "INT2" I R 2950 2600 50
+F13 "INT4" I R 2950 2700 50
+F14 "INT6" I R 2950 2800 50
+F15 "I2C0_SDA" I R 2950 2900 50
+F16 "I2C1_SDA" I R 2950 3000 50
+F17 "INT8" I R 2950 3100 50
+F18 "SPI0_nSS2" I R 2950 3200 50
+F19 "SPI0_nSS3" I R 2950 3300 50
+F20 "SPI0_nSS4" I R 2950 3400 50
+F21 "SPI0_nSS5" I R 2950 3500 50
+F22 "SPI0_nSS6" I R 2950 3600 50
+F23 "SPI0_nSS7" I R 2950 3700 50
+F24 "SPI0_nSS8" I R 2950 3800 50
+F25 "SPIHS_SCK" I L 1700 4050 50
+F26 "SPIHS_MISO" I R 2950 4050 50
+F27 "SPIHS_MOSI" I L 1700 4150 50
+F28 "SPIHS_nSS1" I L 1700 4250 50
+F29 "SPIHS_nSS2" I R 2950 4250 50
 $EndSheet
-Text Label 7200 1950 2    50   ~ 0
+Text Label 1250 3200 2    50   ~ 0
 SPI_nSS1
 Wire Wire Line
-	7200 1950 7650 1950
-Text Label 7200 2150 2    50   ~ 0
+	1250 3200 1700 3200
+Text Label 1250 3400 2    50   ~ 0
 SPI_MISO
 Wire Wire Line
-	7200 2150 7650 2150
-Text Label 7200 2250 2    50   ~ 0
+	1250 3400 1700 3400
+Text Label 1250 3500 2    50   ~ 0
 SPI_MOSI
 Wire Wire Line
-	7200 2250 7650 2250
-Text Label 7200 2050 2    50   ~ 0
+	1250 3500 1700 3500
+Text Label 1250 3300 2    50   ~ 0
 SPI_SCK
 Wire Wire Line
-	7200 2050 7650 2050
-Text Label 9400 1850 0    50   ~ 0
+	1250 3300 1700 3300
+Text Label 3450 3100 0    50   ~ 0
 IO_39
 Wire Wire Line
-	9400 1850 8900 1850
-Text Label 7200 1850 2    50   ~ 0
+	3450 3100 2950 3100
+Text Label 1250 3100 2    50   ~ 0
 IO_38
 Wire Wire Line
-	7200 1850 7650 1850
+	1250 3100 1700 3100
+Wire Notes Line
+	550  550  550  2150
+Wire Notes Line
+	550  2150 3950 2150
+Wire Notes Line
+	3950 2150 3950 550
+Wire Notes Line
+	3950 550  550  550
+Text Notes 3700 2100 0    50   ~ 0
+Radio
+Wire Notes Line
+	550  2300 3950 2300
+Wire Notes Line
+	3950 2300 3950 4800
+Wire Notes Line
+	3950 4800 550  4800
+Wire Notes Line
+	550  4800 550  2300
+Text Notes 3600 4750 0    50   ~ 0
+CAS Bus
+Text Label 950  1150 2    50   ~ 0
+ANT
+Wire Wire Line
+	950  1150 1500 1150
+$Comp
+L ANT-433-SP:ANT-433-SP E1
+U 1 1 5F9A1ADA
+P 1200 5200
+F 0 "E1" H 1285 5229 50  0000 L CNN
+F 1 "ANT-433-SP" H 1285 5138 50  0000 L CNN
+F 2 "radio:XDCR_ANT-433-SP" H 1200 5200 50  0001 L BNN
+F 3 "1.5 mm" H 1200 5200 50  0001 L BNN
+F 4 "Linx" H 1200 5200 50  0001 L BNN "Field4"
+F 5 "1/3/2017" H 1200 5200 50  0001 L BNN "Field5"
+F 6 "Manufacturer Recommendations" H 1200 5200 50  0001 L BNN "Field6"
+	1    1200 5200
+	1    0    0    -1
+$EndComp
+$Comp
+L power:GND #PWR0101
+U 1 1 5F9A1F79
+P 1000 5700
+F 0 "#PWR0101" H 1000 5450 50  0001 C CNN
+F 1 "GND" H 1005 5527 50  0000 C CNN
+F 2 "" H 1000 5700 50  0001 C CNN
+F 3 "" H 1000 5700 50  0001 C CNN
+	1    1000 5700
+	1    0    0    -1
+$EndComp
+Wire Wire Line
+	1100 5300 1000 5300
+Wire Wire Line
+	1000 5300 1000 5400
+Wire Wire Line
+	1100 5700 1000 5700
+Connection ~ 1000 5700
+Wire Wire Line
+	1100 5600 1000 5600
+Connection ~ 1000 5600
+Wire Wire Line
+	1000 5600 1000 5700
+Wire Wire Line
+	1100 5500 1000 5500
+Connection ~ 1000 5500
+Wire Wire Line
+	1000 5500 1000 5600
+Wire Wire Line
+	1100 5400 1000 5400
+Connection ~ 1000 5400
+Wire Wire Line
+	1000 5400 1000 5500
+Text Label 1000 5200 2    50   ~ 0
+ANT
+Wire Wire Line
+	1000 5200 1100 5200
+Wire Notes Line
+	550  4950 550  6000
+Wire Notes Line
+	550  6000 2050 6000
+Wire Notes Line
+	2050 6000 2050 4950
+Wire Notes Line
+	2050 4950 550  4950
+Text Notes 1700 5950 0    50   ~ 0
+Antenna
 $EndSCHEMATC
